File: LineFollower_V5.0/LineFollower_V2.0.kicad_sch (KiCad schematic)
At the start: 20 parts, among them J1 BAT, J3 ICSP, J4 Conn_01x06_MountingPin, J5 Conn_01x10, J6 MotA, J7 MotB, SW1 RESET, SW2 POW, U1 ATmega328P-AU, U2 LM78L05_TO92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

Commit message: upppd
Parts:
- removed C4, C5: 100nF, Capacitor_SMD:C_1206_3216Metric_Pad1.33x1.80mm_HandSolder, symbol Device:C
- removed SW2: POW, symbol Connector_Generic:Conn_01x03
- added J2: Conn_01x05, symbol Connector_Generic:Conn_01x05
- added SW2: SW_SPDT, symbol Switch:SW_SPDT
- C6: footprint (none) -> Capacitor_SMD:C_0805_2012Metric
- J3: footprint (none) -> Connector_PinHeader_2.54mm:PinHeader_2x03_P2.54mm_Vertical
- J5: footprint (none) -> Connector_PinHeader_2.54mm:PinHeader_1x10_P2.54mm_Horizontal
- J6, J7: footprint Connector_PinHeader_2.54mm:PinHeader_1x02_P2.54mm_Horizontal -> Connector_PinHeader_2.54mm:PinHeader_1x02_P2.54mm_Vertical
- R1, R2: footprint (none) -> Resistor_SMD:R_1206_3216Metric
- Y1: value 16MHz -> 20MHz
Connections:
- net 10 is gone; now on net PWMB: U1.14 (~PB2)
- net D8 is gone; now on net BIN1: U1.12 (PB0)
- net D9 is gone; now on net BIN2: U1.13 (~PB1)
- net +5V: now also J2.5 (Pin_5)
- net BIN1: now also U3.16 (BIN2); no longer U1.11 (PD7), U3.17 (BIN1)
- net BIN2: now also U3.17 (BIN1); no longer U1.10 (~PD6), U3.16 (BIN2)
- net Earth: now also SW1.2, J2.4 (Pin_4), SW2.2 (B); no longer D1.1 (K), SW1.1
- net PWMB: no longer U1.9 (~PD5)
- net RESET: now also SW1.1; no longer SW1.2
- net Sensor0: now also J5.8 (Pin_8); no longer J5.6 (Pin_6)
- net Sensor1: now also J5.7 (Pin_7); no longer J5.5 (Pin_5)
- net Sensor2: now also J5.6 (Pin_6); no longer J5.4 (Pin_4)
- net Sensor3: now also J5.5 (Pin_5); no longer J5.3 (Pin_3)
- net Sensor4: now also J5.4 (Pin_4); no longer J5.2 (Pin_2)
- net Sensor5: now also J5.3 (Pin_3); no longer J5.1 (Pin_1)
- net Sensor6: now also J5.2 (Pin_2); no longer J5.8 (Pin_8)
- net Sensor7: now also J5.1 (Pin_1); no longer J5.7 (Pin_7)
- net at J1.2 (Pin_2): now also D1.1 (K), SW2.1 (A)
- net at U3.1 (AO1), U3.2 (AO1): now also J6.1 (Pin_1); no longer J6.2 (Pin_2)
- net at U3.5 (AO2), U3.6 (AO2): now also J6.2 (Pin_2); no longer J6.1 (Pin_1)
- new net D5: J2.1 (Pin_1), U1.9 (~PD5)
- new net D6: J2.2 (Pin_2), U1.10 (~PD6)
- new net D7: J2.3 (Pin_3), U1.11 (PD7)
Other:
- moved on the sheet: J7, U3

Commit message: f
Connections:
- net Earth: now also D1.1 (K)
- net at J1.2 (Pin_2), SW2.1 (A): no longer D1.1 (K)
Other:
- moved on the sheet: SW2
