File: LineFollower_V5.0/LineFollower_V2.0.kicad_pcb (KiCad board)
At the start: 2 copper layers, 15 x 13.6 mm, 20 parts, among them J1 BAT, J3 ICSP, J4 Conn_01x06_MountingPin, J5 Conn_01x10, J6 MotA, J7 MotB, SW1 RESET, SW2 POW, U1 ATmega328P-AU, U2 LM78L05_TO92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

Commit message: upppd
Parts:
- removed C4, C5: 100nF, Capacitor_SMD:C_1206_3216Metric_Pad1.33x1.80mm_HandSolder
- removed U3: TB6612FNG, TB6612FNG:SOP65P760X160-24N
- added J8: BAT, Connector_PinSocket_2.54mm:PinSocket_1x08_P2.54mm_Vertical, F.Cu at (142.1, 96.4)
- added J9: Conn_01x03, Connector_PinSocket_2.54mm:PinSocket_1x08_P2.54mm_Vertical, F.Cu at (142.1, 111.7)
- added REF**: PinHeader_1x05_P2.54mm_Vertical, Connector_PinHeader_2.54mm:PinHeader_1x05_P2.54mm_Vertical, F.Cu at (139.5, 118.2)
- J6: renamed from J7; value MotB -> MotA
- J7: renamed from J6; value MotA -> MotB
- R1: footprint Resistor_SMD:R_1206_3216Metric -> Resistor_SMD:R_0603_1608Metric_Pad0.98x0.95mm_HandSolder
- SW1: moved to F.Cu
- SW2: value POW -> SW_SPDT; footprint Connector_PinHeader_2.54mm:PinHeader_1x03_P2.54mm_Vertical -> Button_Switch_THT:SW_CuK_OS102011MA1QN1_SPDT_Angled
- Y1: value 16MHz -> 20MHz
- moved J5 108.9 mm to (161.4, 89.2)
- moved J1 103.8 mm to (140.8, 101.6), turned to 0 degrees
- moved D1 93.0 mm to (124.7, 90.2), turned to 90 degrees
- moved SW2 86.9 mm to (137.4, 82.4), turned to 180 degrees
- moved R2 86.9 mm to (127.9, 90.3)
- moved J3 86.5 mm to (153.7, 114.6)
- moved C2 86.2 mm to (139.3, 89.0)
- moved C3 86.2 mm to (130.8, 89.0)
- moved U2 86.2 mm to (135.0, 86.9)
- moved J6 80.4 mm to (127.1, 108.5)
- moved J7 80.4 mm to (127.1, 102.2)
- moved Y1 80.4 mm to (146.7, 111.5), turned to 0 degrees
- moved U1 80.1 mm to (153.0, 105.8)
- moved C6 53.5 mm to (144.4, 85.5)
- moved J4 51.8 mm to (156.1, 82.7), turned to -90 degrees
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Connections:
- J1 pad 2: Net-(SW2-Pad2) -> Net-(D1-K)
- J5 pad 1: Sensor5 -> Sensor7
- J5 pad 2: Sensor4 -> Sensor6
- J5 pad 3: Sensor3 -> Sensor5
- J5 pad 4: Sensor2 -> Sensor4
- J5 pad 5: Sensor1 -> Sensor3
- J5 pad 6: Sensor0 -> Sensor2
- J5 pad 7: Sensor7 -> Sensor1
- J5 pad 8: Sensor6 -> Sensor0
- SW1 pad 1: 0V -> RESET
- SW1 pad 2: RESET -> 0V
- SW2 pad 1: 0V -> Net-(D1-K)
- SW2 pad 2: Net-(SW2-Pad2) -> 0V
- U1 pad 10: BIN2 -> D6
- U1 pad 11: BIN1 -> D7
- U1 pad 12: D8 -> BIN1
- U1 pad 13: D9 -> BIN2
- U1 pad 14: 10 -> PWMB
- U1 pad 9: PWMB -> D5
Routing:
- net 0V: track 45.8 -> 221.9 mm, vias 0 -> 1
- net 5V: track 43.5 -> 141.1 mm
- net RESET: track 0.00 -> 50.4 mm, vias 0 -> 1
- net Net-(D1-K): track 0.00 -> 26.9 mm
- net D5: track 0.00 -> 23.7 mm, vias 0 -> 1
- net PWMB: track 9.90 -> 31.7 mm, vias 0 -> 1
- net D6: track 0.00 -> 20.3 mm, vias 0 -> 1
- net RX: track 5.07 -> 24.0 mm, vias 0 -> 1
- net Sensor6: track 0.00 -> 18.3 mm, vias 0 -> 1
- net TX: track 5.32 -> 23.4 mm, vias 0 -> 1
- net Sensor7: track 0.00 -> 17.9 mm, vias 0 -> 1
- net +BATT: track 32.2 -> 15.5 mm, vias 2 -> 0
- net D7: track 0.00 -> 15.6 mm, vias 0 -> 1
- net GND: track 13.9 -> 0.00 mm
- net BIN2: track 15.7 -> 27.6 mm, vias 0 -> 1
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Other:
- board size 15 x 13.6 mm -> 43.5 x 41.2 mm
- board text added: "D2 AIN1 D4 AIN2 D3 PWMA D8 BIN1 D9 BIN2 D10 PWMB"
- board text added: "D5"
- board text added: "D6"
- board text added: "D7"
- board text added: "TB6612FNG MotorDriver"
- board text removed: "CLK 20MHZ ???"
- board text removed: "D10"
- board text removed: "D2-AIN1 D3-PWMA D4-AIN2 D5-PWMB D6-BIN2 D7-BIN1"
- board text removed: "D8"
- board text removed: "D9"

Commit message: f
Parts:
- J2: renamed from REF**; value PinHeader_1x05_P2.54mm_Vertical -> Conn_01x05
- J6: renamed from J7; value MotB -> MotA
- J7: renamed from J6; value MotA -> MotB
Changed lines of the file:
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@@
   (net 34 "Net-(J7-Pin_2)")
   (net 35 "unconnected-(SW2-C-Pad3)")
-  (net 36 "Net-(D1-K)")
+  (net 36 "Net-(J1-Pin_2)")
   (footprint "Connector_PinSocket_2.54mm:PinSocket_1x06_P2.54mm_Vertical" (layer "F.Cu")
     (at 156.1378 82.6872 -90)
@@
       (net 3 "0V"))
     (pad "1" thru_hole rect (at 0 0 180) (size 1.5 2.5) (drill 0.9) (layers "*.Cu" "*.Mask")
-      (net 36 "Net-(D1-K)") (pinfunction "A") (pintype "passive"))
+      (net 36 "Net-(J1-Pin_2)") (pinfunction "A") (pintype "passive"))
     (pad "2" thru_hole oval (at 2 0 180) (size 1.5 2.5) (drill 0.9) (layers "*.Cu" "*.Mask")
       (net 3 "0V") (pinfunction "B") (pintype "passive"))
@@
     (descr "Through hole straight pin header, 1x05, 2.54mm pitch, single row")
     (tags "Through hole pin header THT 1x05 2.54mm single row")
+    (property "Sheetfile" "LineFollower_V2.0.kicad_sch")
+    (property "Sheetname" "")
+    (property "ki_description" "Generic connector, single row, 01x05, script generated (kicad-library-utils/schlib/autogen/connector/)")
+    (property "ki_keywords" "connector")
     (attr through_hole)
-    (fp_text reference "REF**" (at 0 -2.33 90) (layer "F.SilkS") hide
-        (effects (font (size 1 1) (thickness 0.15)))
-    )
-    (fp_text value "PinHeader_1x05_P2.54mm_Vertical" (at 0 12.49 90) (layer "F.Fab")
+    (fp_text reference "J2" (at 0 -2.33 90) (layer "F.SilkS") hide
+        (effects (font (size 1 1) (thickness 0.15)))
+    )
+    (fp_text value "Conn_01x05" (at 0 12.49 90) (layer "F.Fab")
         (effects (font (size 1 1) (thickness 0.15)))
     )
@@
       (stroke (width 0.1) (type solid)) (layer "F.Fab"))
     (pad "1" thru_hole rect (at 0 0 90) (size 1.7 1.7) (drill 1) (layers "*.Cu" "*.Mask")
-      (net 25 "D5"))
+      (net 25 "D5") (pinfunction "Pin_1") (pintype "passive"))
     (pad "2" thru_hole oval (at 0 2.54 90) (size 1.7 1.7) (drill 1) (layers "*.Cu" "*.Mask")
-      (net 26 "D6"))
+      (net 26 "D6") (pinfunction "Pin_2") (pintype "passive"))
     (pad "3" thru_hole oval (at 0 5.08 90) (size 1.7 1.7) (drill 1) (layers "*.Cu" "*.Mask")
-      (net 27 "D7"))
+      (net 27 "D7") (pinfunction "Pin_3") (pintype "passive"))
     (pad "4" thru_hole oval (at 0 7.62 90) (size 1.7 1.7) (drill 1) (layers "*.Cu" "*.Mask")
-      (net 3 "0V"))
+      (net 3 "0V") (pinfunction "Pin_4") (pintype "passive"))
     (pad "5" thru_hole oval (at 0 10.16 90) (size 1.7 1.7) (drill 1) (layers "*.Cu" "*.Mask")
-      (net 4 "5V"))
+      (net 4 "5V") (pinfunction "Pin_5") (pintype "passive"))
     (model "${KICAD6_3DMODEL_DIR}/Connector_PinHeader_2.54mm.3dshapes/PinHeader_1x05_P2.54mm_Vertical.wrl"
       (offset (xyz 0 0 0))
@@
     (property "ki_keywords" "connector")
     (attr through_hole)
-    (fp_text reference "J7" (at -0.02 5.08) (layer "F.SilkS") hide
-        (effects (font (size 1 1) (thickness 0.15)))
-    )
-    (fp_text value "MotB" (at -2.2 1.39 90) (layer "F.SilkS")
+    (fp_text reference "J6" (at -0.02 5.08) (layer "F.SilkS") hide
+        (effects (font (size 1 1) (thickness 0.15)))
+    )
+    (fp_text value "MotA" (at -2.2 1.39 90) (layer "F.SilkS")
         (effects (font (size 1 1) (thickness 0.25)))
     )
@@
     (property "ki_keywords" "connector")
     (attr through_hole)
-    (fp_text reference "J6" (at 2.77 -2.75) (layer "F.SilkS") hide
-        (effects (font (size 1 1) (thickness 0.15)))
-    )
-    (fp_text value "MotA" (at -2.3 1.49 90) (layer "F.SilkS")
+    (fp_text reference "J7" (at 2.77 -2.75) (layer "F.SilkS") hide
+        (effects (font (size 1 1) (thickness 0.15)))
+    )
+    (fp_text value "MotB" (at -2.3 1.49 90) (layer "F.SilkS")
         (effects (font (size 1 1) (thickness 0.25)))
     )
@@
       (net 5 "+BATT") (pinfunction "Pin_1") (pintype "passive"))
     (pad "2" thru_hole oval (at 0 2.54) (size 1.7 1.7) (drill 1) (layers "*.Cu" "*.Mask")
-      (net 36 "Net-(D1-K)") (pinfunction "Pin_2") (pintype "passive"))
+      (net 36 "Net-(J1-Pin_2)") (pinfunction "Pin_2") (pintype "passive"))
     (model "${KICAD6_3DMODEL_DIR}/Connector_PinHeader_2.54mm.3dshapes/PinHeader_1x02_P2.54mm_Vertical.wrl" hide
       (offset (xyz 0 0 0))

Commit message: s
Parts:
- added G***: LOGO, LOGO, B.Cu at (133.6, 103.8)
Other:
- board text added: "A0"
- board text added: "A7"
- board text added: "MotA"
- board text added: "MotB"
